File: V1.0/Alchemy.kicad_pcb (KiCad board)
At the start: 4 copper layers, 55 x 85 mm, 66 parts, among them J1 Conn_02x20_Odd_Even, J2 USB_C_Receptacle_USB2.0, J3 USB_C_Receptacle_USB2.0, J4 Conn_01x03, J5 Conn_01x03, U1 CH32V203C8T6, U2 LM5164DDA, U3 CH340G, U4 AMS1117-3.3, U5 MT9700, U6 MT9700, U7 MT9700, Y1 12Mz, Y2 8MHz

Commit message: Updated BOM
Parts:
- R11: value 1K -> 4.7K
- R13: value 1k -> 4.7K
Changed lines of the file:
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@@
       (effects (font (size 1 1) (thickness 0.15)))
     )
-    (fp_text value "1k" (at 0 1.65) (layer "F.Fab") hide
+    (fp_text value "4.7K" (at 0 1.65) (layer "F.Fab") hide
       (effects (font (size 1 1) (thickness 0.15)))
     )
@@
       (effects (font (size 1 1) (thickness 0.15)))
     )
-    (fp_text value "1K" (at 0 1.65 90) (layer "F.Fab") hide
-      (effects (font (size 1 1) (thickness 0.15)))
-    )
+    (fp_text value "4.7K" (at 0 1.65 90) (layer "F.Fab") hide
+      (effects (font (size 1 1) (thickness 0.15)))
+    )
