File: V1.0/Alchemy.kicad_sch (KiCad schematic)
At the start: 66 parts, among them J1 Conn_02x20_Odd_Even, J2 USB_C_Receptacle_USB2.0, J3 USB_C_Receptacle_USB2.0, J4 Conn_01x03, J5 Conn_01x03, U1 CH32V203C8T6, U2 LM5164DDA, U3 CH340G, U4 AMS1117-3.3, U5 MT9700, U6 MT9700, U7 MT9700, Y1 12Mz, Y2 8MHz

Commit message: Updated BOM
Parts:
- R11: value 1K -> 4.7K
- R13: value 1k -> 4.7K
Changed lines of the file:
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@@
       (effects (font (size 1.27 1.27)) (justify left))
     )
-    (property "Value" "1K" (id 1) (at 213.36 247.6499 0)
+    (property "Value" "4.7K" (id 1) (at 213.36 247.6499 0)
       (effects (font (size 1.27 1.27)) (justify left))
     )
@@
     (in_bom yes) (on_board yes)
     (property "Reference" "R13" (id 0) (at 256.54 251.46 90))
-    (property "Value" "1k" (id 1) (at 256.54 254 90))
+    (property "Value" "4.7K" (id 1) (at 256.54 254 90))
     (property "Footprint" "Resistor_SMD:R_0805_2012Metric" (id 2) (at 256.54 258.318 90)
       (effects (font (size 1.27 1.27)) hide)
@@
     )
     (path "/1447db99-25e3-4c56-9879-a4748f02e532"
-      (reference "R11") (unit 1) (value "1K") (footprint "Resistor_SMD:R_0805_2012Metric")
+      (reference "R11") (unit 1) (value "4.7K") (footprint "Resistor_SMD:R_0805_2012Metric")
     )
     (path "/ccb50aa5-41d1-4e5d-b1ae-a08b0048ef60"
@@
     )
     (path "/9407fd27-b436-4d40-9a01-76e07eca19b2"
-      (reference "R13") (unit 1) (value "1k") (footprint "Resistor_SMD:R_0805_2012Metric")
+      (reference "R13") (unit 1) (value "4.7K") (footprint "Resistor_SMD:R_0805_2012Metric")
     )
     (path "/eb8ebd2f-7cab-40c1-a27a-7a0c1d8ce7d1"
