File: V2.0A/Alchemy.kicad_sch (KiCad schematic)
At the start: 65 parts, among them J1 Conn_02x20_Odd_Even, J2 USB_C_Receptacle_USB2.0, J3 USB_C_Receptacle_USB2.0, J4 Conn_01x03, J5 Conn_01x03, J6 Conn_01x02, J7 Conn_01x02, J8 Conn_01x02, J9 Conn_01x03, U1 CH32V203C8T6, U2 LM5164DDA, U3 CH213K, U4 AMS1117-3.3, U5 CH213K, U6 MT9700, Y2 8MHz

Commit message: Updated Nano-FOC firmware
Other:
- note added: "19.09.2025"
- note added: "Alchemy V2.0A"
- note removed: "29.12.2023"
- note removed: "Alchemy V1.0"
Changed lines of the file:
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@@
     (stroke (width 0) (type default) (color 0 0 0 0))
   )
-  (text "29.12.2023" (at 332.74 280.67 0)
+  (text "19.09.2025" (at 332.74 280.67 0)
     (effects (font (size 1.27 1.27)) (justify left bottom))
   )
-  (text "Alchemy V1.0" (at 312.42 278.13 0)
+  (text "Alchemy V2.0A" (at 312.42 278.13 0)
     (effects (font (size 1.27 1.27)) (justify left bottom))
   )
